File: H-Bridge.kicad_pcb (KiCad board)
At the start: 2 copper layers, 22 parts, among them J1 Conn_01x04, J2 Screw_Terminal_01x02, J3 Screw_Terminal_01x02, Q1 Q_NPN_CBE, Q2 Q_PNP_CBE, Q3 Q_NPN_CBE, Q4 Q_PNP_CBE, Q5 Q_NMOS_GDS, Q6 Q_NMOS_GDS, Q7 Q_NMOS_GDS, Q8 Q_NMOS_GDS

Commit message: 1
Other:
- board text added: "+"
- board text added: "+12V"
- board text added: "-"
- board text added: "1"
- board text added: "2"
- board text added: "Input"
- board text added: "Output"
- board text added: "S-"
Changed lines of the file:
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@@
   (general
     (thickness 1.6)
-    (drawings 0)
+    (drawings 8)
     (tracks 90)
     (zones 0)
@@
     (solder_mask_min_width 0.25)
     (aux_axis_origin 0 0)
-    (visible_elements FFFFFF7F)
+    (visible_elements 7FFFFFFF)
     (pcbplotparams
       (layerselection 0x010fc_ffffffff)
@@
     (tags connector)
     (attr virtual)
-    (fp_text reference J3 (at 3.175 -3.81 90) (layer F.SilkS)
+    (fp_text reference J3 (at 10.16 -1.905) (layer F.SilkS)
       (effects (font (size 1 1) (thickness 0.15)))
     )
@@
     (tags connector)
     (attr virtual)
-    (fp_text reference J2 (at 3.175 -3.81 90) (layer F.SilkS)
+    (fp_text reference J2 (at 10.16 0 180) (layer F.SilkS)
       (effects (font (size 1 1) (thickness 0.15)))
     )
@@
     )
   )
+  (gr_text +12V (at 111.76 88.265 -90) (layer F.SilkS)
+    (effects (font (size 1 1) (thickness 0.25)))
+  )
+  (gr_text 1 (at 111.76 92.075 -90) (layer F.SilkS)
+    (effects (font (size 1 1) (thickness 0.25)))
+  )
+  (gr_text 2 (at 111.76 94.615 -90) (layer F.SilkS)
+    (effects (font (size 1 1) (thickness 0.25)))
+  )
+  (gr_text S- (at 111.76 97.155 -90) (layer F.SilkS)
+    (effects (font (size 1 1) (thickness 0.25)))
+  )
+  (gr_text Input (at 114.3 109.22 -90) (layer F.SilkS)
+    (effects (font (size 1.5 1.5) (thickness 0.3)))
+  )
+  (gr_text - (at 109.855 116.84 -90) (layer F.SilkS)
+    (effects (font (size 2.5 2.5) (thickness 0.3)))
+  )
+  (gr_text + (at 109.855 101.6 -90) (layer F.SilkS)
+    (effects (font (size 2.5 2.5) (thickness 0.3)))
+  )
+  (gr_text Output (at 219.71 109.22 90) (layer F.SilkS)
+    (effects (font (size 1.5 1.5) (thickness 0.3)))
+  )
   (segment (start 178.435 89.535) (end 178.435 107.315) (width 2) (layer B.Cu) (net 1))

Commit message: 1
Parts:
- removed the D3 at (190.5, 115.6)
- removed the Q2 at (148.6, 94.6)
- removed the Q4 at (148.6, 123.2)
- removed the R6 at (167.6, 95.9)
- added D1: D, Diode_THT:D_DO-15_P12.70mm_Horizontal, F.Cu at (198.1, 93.3)
- added R10: 100k, Resistor_THT:R_Axial_DIN0207_L6.3mm_D2.5mm_P10.16mm_Horizontal, F.Cu at (202.6, 96.5)
- added R11: 100k, Resistor_THT:R_Axial_DIN0207_L6.3mm_D2.5mm_P10.16mm_Horizontal, F.Cu at (212.7, 120.7)
- added R8: 100k, Resistor_THT:R_Axial_DIN0207_L6.3mm_D2.5mm_P10.16mm_Horizontal, F.Cu at (181.0, 120.7)
- moved R7 24.3 mm to (170.8, 96.5), turned to 0 degrees
- moved D3 17.5 mm to (185.4, 110.5), turned to 0 degrees
- moved D2 12.7 mm to (185.4, 123.8), turned to 0 degrees
- moved R3 12.3 mm to (140.3, 94.6), turned to 270 degrees
- moved R4 12.3 mm to (140.3, 121.9), turned to 90 degrees
- moved R5 11.9 mm to (166.4, 101.6)
- moved R6 11.9 mm to (166.4, 114.9)
- moved Q2 6.35 mm to (148.0, 112.4)
- moved J1 6.35 mm to (114.9, 97.2)
- moved J3 6.35 mm to (116.2, 106.0)
- moved Q1 6.35 mm to (148.6, 104.1)
- moved R1 6.35 mm to (133.3, 104.8)
- moved R2 6.35 mm to (133.3, 111.8)
- renumbered D1 to D3, Q3 to Q2, Q5 to Q3, Q6 to Q4, Q7 to Q5, Q8 to Q6, R8 to R6
Connections:
- D3 pad 2: Net-(D1-Pad2) -> Net-(D3-Pad2)
- Q2 pad 2: Net-(Q3-Pad2) -> Net-(Q2-Pad2)
- Q2 pad 3: Net-(Q3-Pad3) -> Net-(Q2-Pad3)
- Q3 pad 1: Net-(Q5-Pad1) -> Net-(Q3-Pad1)
- Q4 pad 1: Net-(Q6-Pad1) -> Net-(Q4-Pad1)
- Q5 pad 1: Net-(Q6-Pad1) -> Net-(Q4-Pad1)
- Q6 pad 1: Net-(Q5-Pad1) -> Net-(Q3-Pad1)
- R2 pad 1: Net-(Q3-Pad2) -> Net-(Q2-Pad2)
- R3 pad 1: Net-(Q1-Pad2) -> Net-(Q1-Pad3)
- R3 pad 2: GNDS -> Net-(Q1-Pad2)
- R4 pad 1: Net-(Q3-Pad2) -> Net-(Q2-Pad3)
- R4 pad 2: GNDS -> Net-(Q2-Pad2)
- R5 pad 1: Net-(Q6-Pad1) -> Net-(Q3-Pad1)
- R5 pad 2: Net-(Q3-Pad3) -> Net-(Q1-Pad3)
- R6 pad 1: Net-(Q5-Pad1) -> Net-(Q4-Pad1)
- R6 pad 2: Net-(Q1-Pad3) -> Net-(Q2-Pad3)
- R7 pad 1: Net-(Q6-Pad1) -> Net-(Q3-Pad1)
- R7 pad 2: GNDS -> Net-(D1-Pad2)
Routing:
- net Net-(Q3-Pad1): track 0.00 -> 83.0 mm
- net Net-(Q6-Pad1): track 75.6 -> 0.00 mm
- net Net-(Q5-Pad1): track 73.8 -> 0.00 mm
- net Net-(Q4-Pad1): track 0.00 -> 72.8 mm
- net Net-(Q3-Pad2): track 36.0 -> 0.00 mm
- net Net-(Q3-Pad3): track 21.4 -> 0.00 mm
- net Net-(Q1-Pad2): track 36.5 -> 16.0 mm
- net Net-(Q2-Pad3): track 0.00 -> 19.2 mm
- net Net-(Q2-Pad2): track 0.00 -> 15.4 mm
- net GND: track 118.6 -> 126.9 mm
- net Net-(D3-Pad2): track 60.1 -> 68.0 mm
- net VCC: track 114.8 -> 108.4 mm
- net Net-(D1-Pad2): track 94.5 -> 99.5 mm

Commit message: 1
Parts:
- added Q3: Q_NPN_CBE, Package_TO_SOT_THT:TO-92_Inline, F.Cu at (158.8, 105.4)
- added Q4: Q_PNP_CBE, Package_TO_SOT_THT:TO-92_Inline, F.Cu at (158.8, 97.8)
- added Q5: Q_NPN_CBE, Package_TO_SOT_THT:TO-92_Inline, F.Cu at (158.8, 121.9)
- added Q6: Q_PNP_CBE, Package_TO_SOT_THT:TO-92_Inline, F.Cu at (158.8, 114.3)
- R1: value 100 -> 1k
- R2: value 100 -> 100k
- R4: value 1k -> 100k
- R5, R6: value 100 -> 10k
- moved R5 21.7 mm to (145.4, 95.9), turned to 270 degrees
- moved R6 21.1 mm to (145.4, 112.4), turned to 270 degrees
- moved R2 17.3 mm to (140.3, 95.9), turned to 270 degrees
- moved R3 12.5 mm to (135.3, 106.0), turned to 90 degrees
- moved Q2 11.1 mm to (152.4, 122.6), turned to 90 degrees
- moved R4 9.53 mm to (140.3, 112.4), turned to 270 degrees
- moved R1 7.85 mm to (135.3, 112.4), turned to 270 degrees
- moved Q1 4.26 mm to (152.4, 106.0)
- moved D3 1.91 mm to (185.4, 112.4)
- renumbered Q6 to Q10, Q3 to Q7, Q4 to Q8, Q5 to Q9, R11 to R10, R10 to R9
Connections:
- Q1 pad 1: +12V -> Net-(Q1-Pad1)
- Q1 pad 3: Net-(Q1-Pad3) -> GNDS
- Q10 pad 1: Net-(Q3-Pad1) -> Net-(Q10-Pad1)
- Q2 pad 1: +12V -> Net-(Q2-Pad1)
- Q2 pad 3: Net-(Q2-Pad3) -> GNDS
- Q7 pad 1: Net-(Q3-Pad1) -> Net-(Q10-Pad1)
- Q8 pad 1: Net-(Q4-Pad1) -> Net-(Q5-Pad3)
- Q9 pad 1: Net-(Q4-Pad1) -> Net-(Q5-Pad3)
- R1 pad 1: Net-(Q1-Pad2) -> Net-(J1-Pad2)
- R1 pad 2: Net-(J1-Pad3) -> Net-(Q2-Pad2)
- R10 pad 1: Net-(Q3-Pad1) -> Net-(Q10-Pad1)
- R2 pad 1: Net-(Q2-Pad2) -> +12V
- R2 pad 2: Net-(J1-Pad2) -> Net-(Q1-Pad2)
- R3 pad 1: Net-(Q1-Pad3) -> Net-(Q1-Pad2)
- R3 pad 2: Net-(Q1-Pad2) -> Net-(J1-Pad3)
- R4 pad 1: Net-(Q2-Pad3) -> +12V
- R5 pad 1: Net-(Q3-Pad1) -> +12V
- R5 pad 2: Net-(Q1-Pad3) -> Net-(Q1-Pad1)
- R6 pad 1: Net-(Q4-Pad1) -> +12V
- R6 pad 2: Net-(Q2-Pad3) -> Net-(Q2-Pad1)
- R7 pad 1: Net-(Q3-Pad1) -> Net-(Q10-Pad1)
- R8 pad 1: Net-(Q4-Pad1) -> Net-(Q5-Pad3)
- R9 pad 1: Net-(Q4-Pad1) -> Net-(Q5-Pad3)
Routing:
- net Net-(Q10-Pad1): track 0.00 -> 92.3 mm
- net Net-(Q5-Pad3): track 0.00 -> 84.2 mm
- net Net-(Q3-Pad1): track 83.0 -> 0.00 mm
- net Net-(Q4-Pad1): track 72.8 -> 0.00 mm
- net +12V: track 52.0 -> 92.9 mm
- net Net-(Q2-Pad1): track 0.00 -> 25.1 mm
- net Net-(Q1-Pad1): track 0.00 -> 23.8 mm
- net Net-(Q2-Pad3): track 19.2 -> 0.00 mm
- net Net-(Q1-Pad3): track 19.2 -> 0.00 mm
- net Net-(D3-Pad2): track 68.0 -> 58.6 mm
- net Net-(D1-Pad2): track 99.5 -> 90.2 mm
- net Net-(J1-Pad2): track 20.6 -> 27.7 mm
- net Net-(J1-Pad3): track 16.1 -> 21.9 mm
- net Net-(Q2-Pad2): track 15.4 -> 19.9 mm
- net Net-(Q1-Pad2): track 16.0 -> 19.9 mm
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- added copper zone on B.Cu, net GND
- added copper zone on B.Cu, net Net-(D1-Pad2)
- added copper zone on B.Cu, net Net-(D3-Pad2)
- added copper zone on B.Cu, net VCC
Other:
- board text removed: "-"
