File: H-Bridge.kicad_pcb (KiCad board)
At the start: 2 copper layers, 16 parts, among them J1 Conn_01x03, J2 Screw_Terminal_01x02, J3 Screw_Terminal_01x02, Q1 Q_NMOS_GDS, Q2 Q_NMOS_GDS, Q3 Q_NMOS_GDS, Q4 Q_NMOS_GDS, U1 IRS2181, U2 IRS2181

Commit message: 1
Parts:
- added REF**: , Connector_Wire:SolderWire-0.5sqmm_1x01_D0.9mm_OD2.1mm, F.Cu at (129.5, 86.4)
- added REF**: , Connector_Wire:SolderWire-0.5sqmm_1x01_D0.9mm_OD2.1mm, F.Cu at (129.5, 80.8)
- REF**: value SolderWire-0.5sqmm_1x01_D0.9mm_OD2.1mm -> (none)
Routing:
- net Net-(Q3-Pad1): track 76.0 -> 65.9 mm
