File: H-Bridge.kicad_pcb (KiCad board)
At the start: 2 copper layers, 18 parts, among them J1 Conn_01x03, J2 Screw_Terminal_01x02, J3 Screw_Terminal_01x02, Q1 Q_NMOS_GDS, Q2 Q_NMOS_GDS, Q3 Q_NMOS_GDS, Q4 Q_NMOS_GDS, U1 IRS2181, U2 IRS2181

Commit message: 1
Parts:
- removed REF** (x3): , Connector_Wire:SolderWire-0.5sqmm_1x01_D0.9mm_OD2.1mm
- added C4: 0.1u, Capacitor_SMD:C_0805_2012Metric, F.Cu at (202.2, 89.3)
- added C5: 0.1u, Capacitor_SMD:C_0805_2012Metric, F.Cu at (190.0, 100.1)
- added D3: 18V, Diode_SMD:D_SOD-323, F.Cu at (190.5, 84.3)
- C2, C3: footprint Capacitor_THT:CP_Radial_D10.0mm_P5.00mm -> Capacitor_SMD:C_1206_3216Metric
- D1, D2: footprint Diode_THT:D_DO-34_SOD68_P10.16mm_Horizontal -> Diode_SMD:D_SOD-123
- R1: footprint Resistor_THT:R_Axial_DIN0207_L6.3mm_D2.5mm_P10.16mm_Horizontal -> Resistor_SMD:R_1206_3216Metric
- U1, U2: footprint Package_DIP:DIP-8_W7.62mm -> Package_SO:SOIC-8_3.9x4.9mm_P1.27mm
- moved D2 89.9 mm to (201.7, 100.1)
- moved U1 80.7 mm to (196.1, 89.4)
- moved D1 79.3 mm to (190.5, 89.4), turned to 270 degrees
- moved J2 79.0 mm to (183.9, 81.8)
- moved R1 77.8 mm to (230.1, 95.1)
- moved J1 77.4 mm to (183.4, 97.0), turned to 0 degrees
- moved Q3 77.3 mm to (227.1, 82.8)
- moved Q1 76.3 mm to (210.8, 82.8)
- moved U2 76.0 mm to (196.1, 100.1)
- moved C2 75.8 mm to (195.1, 82.3)
- moved J3 74.7 mm to (235.7, 99.1)
- moved C3 74.6 mm to (197.1, 107.2)
- moved C1 74.1 mm to (212.9, 92.5)
- moved Q2 70.1 mm to (232.2, 106.7)
- moved Q4 69.1 mm to (215.9, 106.7)
Routing:
- net Net-(Q3-Pad1): track 65.9 -> 40.8 mm
- net OUT_B: track 53.8 -> 34.8 mm, vias 0 -> 1
- net Net-(C3-Pad1): track 24.8 -> 8.90 mm
- net Net-(Q4-Pad1): track 42.0 -> 26.5 mm, vias 0 -> 1
- net SIG_B: track 40.0 -> 25.9 mm
- net Net-(Q2-Pad1): track 50.2 -> 40.6 mm, vias 0 -> 2
- net Net-(Q1-Pad1): track 27.8 -> 20.1 mm
- net Net-(C2-Pad1): track 14.9 -> 8.88 mm
- net OUT_A: track 43.7 -> 38.0 mm, vias 0 -> 2
- net SIG_A: track 26.2 -> 20.9 mm
- net GND: vias 0 -> 5
- added copper zone on B.Cu, net OUT_A
- added copper zone on F.Cu, net OUT_B
- removed copper zone on F.Cu, net OUT_A
- removed copper zone on B.Cu, net OUT_B
Other:
- net class Default: clearance 1 -> 0.2
- rule pad_to_mask_clearance: 0.051 -> 0
- rule trace_clearance: 1 -> 0.2

Commit message: Add JLCPCB Files
Parts:
- J1: value Conn_01x03 -> Conn_01x04; footprint Connector_PinSocket_2.54mm:PinSocket_1x03_P2.54mm_Vertical -> Connector_PinSocket_2.54mm:PinSocket_1x04_P2.54mm_Vertical
